File: output/pcbs/left.kicad_pcb (KiCad board)
At the start: 2 copper layers, 146.8 x 123.8 mm, 65 parts

Commit message: adjusted small changes, made right board
Parts:
- added D31: , ComboDiode, F.Cu at (290.0, -14.0)
- added D32: , ComboDiode, F.Cu at (290.0, -33.0)
- added D33: , ComboDiode, F.Cu at (290.0, -52.0)
- added D34: , ComboDiode, F.Cu at (290.0, -71.0)
- added D35: , ComboDiode, F.Cu at (271.0, -14.0)
- added D36: , ComboDiode, F.Cu at (271.0, -33.0)
- added D37: , ComboDiode, F.Cu at (271.0, -52.0)
- added D38: , ComboDiode, F.Cu at (271.0, -71.0)
- added D39: , ComboDiode, F.Cu at (252.0, -7.00)
- added D40: , ComboDiode, F.Cu at (252.0, -26.0)
- added D41: , ComboDiode, F.Cu at (252.0, -45.0)
- added D42: , ComboDiode, F.Cu at (252.0, -64.0)
- added D43: , ComboDiode, F.Cu at (252.0, -83.0)
- added D44: , ComboDiode, F.Cu at (233.0, -12.0)
- added D45: , ComboDiode, F.Cu at (233.0, -31.0)
- added D46: , ComboDiode, F.Cu at (233.0, -50.0)
- added D47: , ComboDiode, F.Cu at (233.0, -69.0)
- added D48: , ComboDiode, F.Cu at (233.0, -88.0)
- added D49: , ComboDiode, F.Cu at (214.0, -6.00)
- added D50: , ComboDiode, F.Cu at (214.0, -25.0)
- added D51: , ComboDiode, F.Cu at (214.0, -44.0)
- added D52: , ComboDiode, F.Cu at (214.0, -63.0)
- added D53: , ComboDiode, F.Cu at (214.0, -82.0)
- added D54: , ComboDiode, F.Cu at (195.0, -23.0)
- added D55: , ComboDiode, F.Cu at (195.0, -42.0)
- added D56: , ComboDiode, F.Cu at (195.0, -61.0)
- added D57: , ComboDiode, F.Cu at (195.0, -80.0)
- added D58: , ComboDiode, F.Cu at (175.0, -28.0)
- added D59: , ComboDiode, F.Cu at (193.9, -1.45)
- added D60: , ComboDiode, F.Cu at (167.3, -3.86)
- added ENC1: RollerEncoder_Panasonic_EVQWGD001, Panasonic_EVQWGD001, F.Cu at (114.5, -52.0)
- added S31: , PG1350, F.Cu at (290.0, -19.0)
- added S32: , PG1350, F.Cu at (290.0, -38.0)
- added S33: , PG1350, F.Cu at (290.0, -57.0)
- added S34: , PG1350, F.Cu at (290.0, -76.0)
- added S35: , PG1350, F.Cu at (271.0, -19.0)
- added S36: , PG1350, F.Cu at (271.0, -38.0)
- added S37: , PG1350, F.Cu at (271.0, -57.0)
- added S38: , PG1350, F.Cu at (271.0, -76.0)
- added S39: , PG1350, F.Cu at (252.0, -12.0)
- added S40: , PG1350, F.Cu at (252.0, -31.0)
- added S41: , PG1350, F.Cu at (252.0, -50.0)
- added S42: , PG1350, F.Cu at (252.0, -69.0)
- added S43: , PG1350, F.Cu at (252.0, -88.0)
- added S44: , PG1350, F.Cu at (233.0, -17.0)
- added S45: , PG1350, F.Cu at (233.0, -36.0)
- added S46: , PG1350, F.Cu at (233.0, -55.0)
- added S47: , PG1350, F.Cu at (233.0, -74.0)
- added S48: , PG1350, F.Cu at (233.0, -93.0)
- added S49: , PG1350, F.Cu at (214.0, -11.0)
- added S50: , PG1350, F.Cu at (214.0, -30.0)
- added S51: , PG1350, F.Cu at (214.0, -49.0)
- added S52: , PG1350, F.Cu at (214.0, -68.0)
- added S53: , PG1350, F.Cu at (214.0, -87.0)
- added S54: , PG1350, F.Cu at (195.0, -28.0)
- added S55: , PG1350, F.Cu at (195.0, -47.0)
- added S56: , PG1350, F.Cu at (195.0, -66.0)
- added S57: , PG1350, F.Cu at (195.0, -85.0)
- added S58: , PG1350, F.Cu at (175.0, -33.0)
- added S59: , PG1350, F.Cu at (192.3, -6.20)
- added S60: , PG1350, F.Cu at (172.1, -5.41)
- moved T1 30.0 mm to (132.2, -76.0), turned to -92.5 degrees
- moved B1 26.2 mm to (130.5, -66.0), turned to -92.5 degrees
- moved JST1 10.6 mm to (128.5, -56.0), turned to 356 degrees
- moved OLED1 8.20 mm to (122.5, -65.5), turned to 261.7 degrees
- moved MCU1 4.27 mm to (118.0, -78.5), turned to 261.7 degrees
Connections:
- D1 pad 1: P011 -> P020
- D10 pad 1: P011 -> P020
- D11 pad 1: P100 -> P017
- D12 pad 1: P024 -> P008
- D13 pad 1: P022 -> P006
- D14 pad 1: P104 -> P022
- D15 pad 1: P011 -> P020
- D16 pad 1: P100 -> P017
- D17 pad 1: P024 -> P008
- D18 pad 1: P022 -> P006
- D19 pad 1: P104 -> P022
- D2 pad 1: P100 -> P017
- D20 pad 1: P011 -> P020
- D21 pad 1: P100 -> P017
- D22 pad 1: P024 -> P008
- D23 pad 1: P022 -> P006
- D24 pad 1: P011 -> P020
- D25 pad 1: P100 -> P017
- D26 pad 1: P024 -> P008
- D27 pad 1: P022 -> P006
- D28 pad 1: P100 -> P017
- D29 pad 1: P104 -> P022
- D3 pad 1: P024 -> P008
- D30 pad 1: P104 -> P022
- D4 pad 1: P022 -> P006
- D5 pad 1: P011 -> P020
- D6 pad 1: P100 -> P017
- D7 pad 1: P024 -> P008
- D8 pad 1: P022 -> P006
- D9 pad 1: P104 -> P022
- OLED1 pad 3: P020 -> P100
- OLED1 pad 4: P017 -> P024
- S1 pad 1: P031 -> P115
- S10 pad 1: P115 -> P111
- S11 pad 1: P115 -> P111
- S12 pad 1: P115 -> P111
- S13 pad 1: P115 -> P111
- S14 pad 1: P113 -> P010
- S15 pad 1: P113 -> P010
- S16 pad 1: P113 -> P010
- S17 pad 1: P113 -> P010
- S18 pad 1: P113 -> P010
- S19 pad 1: P111 -> P009
- S2 pad 1: P031 -> P115
- S20 pad 1: P111 -> P009
- S21 pad 1: P111 -> P009
- S22 pad 1: P111 -> P009
- S23 pad 1: P111 -> P009
- S24 pad 1: P010 -> P011
- S25 pad 1: P010 -> P011
- S26 pad 1: P010 -> P011
- S27 pad 1: P010 -> P011
- S28 pad 1: P009 -> P104
- S29 pad 1: P010 -> P011
- S3 pad 1: P031 -> P115
- S30 pad 1: P009 -> P104
- S4 pad 1: P031 -> P115
- S5 pad 1: P002 -> P113
- S6 pad 1: P002 -> P113
- S7 pad 1: P002 -> P113
- S8 pad 1: P002 -> P113
- S9 pad 1: P115 -> P111
- T1 pad 1: VCC -> pos

Commit message: updates to PCBS. some edits but mostly done PCBs
Parts:
- removed D31, D32, D33, D34, D35, D36, D37, D38, D39, D40, D41, D42, D43, D44, D45, D46, D47, D48, D49, D50, D51, D52, D53, D54, D55, D56, D57, D58, D59, D60: , ComboDiode
- removed S31, S32, S33, S34, S35, S36, S37, S38, S39, S40, S41, S42, S43, S44, S45, S46, S47, S48, S49, S50, S51, S52, S53, S54, S55, S56, S57, S58, S59, S60: , PG1350
- added ?: , HOLE_M2_TH, F.Cu at (25.0, -90.0)
- added ?: , HOLE_M2_TH, F.Cu at (5.00, -7.00)
- added ?: , HOLE_M2_TH, F.Cu at (9.50, -48.0)
- added ?: , HOLE_M2_TH, F.Cu at (66.5, -45.5)
- added ?: , HOLE_M2_TH, F.Cu at (64.0, -3.00)
- added ?: , HOLE_M2_TH, F.Cu at (125.0, 11.0)
- added ?: , HOLE_M2_TH, F.Cu at (107.0, -95.0)
- added ?: , HOLE_M2_TH, F.Cu at (130.0, -37.0)
