File: output/pcbs/right.kicad_pcb (KiCad board)
At the start: 2 copper layers, 146.8 x 123.8 mm, 66 parts

Commit message: updates to PCBS. some edits but mostly done PCBs
Parts:
- added ?: , HOLE_M2_TH, F.Cu at (265.0, -90.0)
- added ?: , HOLE_M2_TH, F.Cu at (285.0, -7.00)
- added ?: , HOLE_M2_TH, F.Cu at (280.5, -48.0)
- added ?: , HOLE_M2_TH, F.Cu at (223.5, -45.5)
- added ?: , HOLE_M2_TH, F.Cu at (226.0, -3.00)
- added ?: , HOLE_M2_TH, F.Cu at (165.0, 11.0)
- added ?: , HOLE_M2_TH, F.Cu at (183.0, -95.0)
- added ?: , HOLE_M2_TH, F.Cu at (160.0, -37.0)
- moved OLED1 12.7 mm to (180.0, -67.5), turned to -81.7 degrees
- moved ENC1 2.06 mm to (176.0, -50.0), turned to -180 degrees
- turned MCU1 to -81.7 degrees
